Commit message: Add LiDAR/IMU + Phase 5 mapping pipeline; make the rover drivable; consolidate docs
Simulation (rover_simulation)
- Add a gpu_lidar (/scan, 10 Hz, frame lidar_link) and an imu (/imu/data, 50 Hz)
  to the inlined rover in lunar_terrain.world, plus the gz-sim-imu-system plugin.
- Bridge /scan and /imu/data in bridge.yaml. Mirror the sensors + a new imu_link
  in rover.urdf.xacro (kept in sync; world file is authoritative at runtime).
- Fix terrain collision: DART ignores <heightmap> collision and DART+ODE trimesh
  collision segfaults, so the ground is now a flat box (top z 0.375 m, mu 0.9) with
  a matching flat plane visual. Rock models keep their own collisions. Rover spawn
  0.38 -> 0.42. scripts/heightmap_to_collision_obj.py + terrain_collision.obj kept
  for a future Bullet-physics contour terrain.

Sensors (sensor_pkg)
- Rewrite encoder_processor with real differential-drive kinematics: wheel-angle
  deltas scaled by wheel_radius, heading integrated from (d_right-d_left)/
  wheel_separation, yaw quaternion + twist published. New pure module
  diff_drive_odometry.py.
- Remove doubled shebangs in imu_processor / lidar_processor.

Mapping (mapping_pkg) - Phase 5
- occupancy_grid_node: log-odds occupancy grid from /scan + TF -> /map, static
  map->odom TF.
- terrain_classifier_node: flat/rocky/crater/obstacle -> /terrain_map + RViz
  markers; periodic snapshot to results/terrain_maps/latest.npz.
- grid_utils.py, terrain_storage.py, mapping.launch.py, params, rviz config.

Tests
- tests/test_grid_utils.py, tests/test_diff_drive_odometry.py (13 tests, CI-safe).

Docs
- Consolidate to two: README.md (guidelines, architecture, setup, run, interfaces,
  assumptions/constraints, Phase 6-12 plan) and docs/PROGRESS.md (status, what was
  done, known issues, next steps, handoff notes).
- Known issue recorded: terrain classifier over-triggers craters; needs
  mapping_params.yaml tuning.

Cleanup
- Remove dead/superseded: scratch/, rover_simulation/models/, setup.py +
  pybullet_sim.py + odom_to_tf.py + rover_teleop.py, unused terrain/rock textures,
  generate_terrain_mesh.py / generate_textures.py / check_scipy.py / drive_test.sh
  / test_physics.sh, the pre-migration roadmap HTML, Humble-era teammate scratch
  files, per-directory READMEs, gazebo_params.yaml, and commented cruft in
  rover_simulation CMakeLists/package.xml.

File: src/rover_simulation/urdf/rover.urdf.xacro (robot description, xacro)
@@ -276,4 +276,84 @@
     <xacro:cylinder_inertia m="0.3" r="0.05" l="0.06"/>
   </link>
+  <!-- ═══════════════════════════════════════════════════════════════════════
+       IMU MOUNT — small module on the chassis, just above centre
+  ═══════════════════════════════════════════════════════════════════════════ -->
+  <joint name="imu_joint" type="fixed">
+    <parent link="base_link"/>
+    <child link="imu_link"/>
+    <origin xyz="0 0 0.07" rpy="0 0 0"/>
+  </joint>
+  <link name="imu_link">
+    <visual>
+      <origin xyz="0 0 0" rpy="0 0 0"/>
+      <geometry>
+        <box size="0.04 0.04 0.02"/>
+      </geometry>
+      <material name="dark_grey"/>
+    </visual>
+    <xacro:box_inertia m="0.05" x="0.04" y="0.04" z="0.02"/>
+  </link>
+  <!-- ═══════════════════════════════════════════════════════════════════════
+       SENSORS — LiDAR + IMU.
+       NOTE: at runtime the simulation loads the rover *inlined* in
+       lunar_terrain.world, which carries its own copies of these sensor
+       blocks. These <gazebo> blocks exist only so a future
+       `xacro rover.urdf.xacro | gz sdf -p -` regeneration stays in sync.
+  ═══════════════════════════════════════════════════════════════════════════ -->
+  <gazebo reference="lidar_link">
+    <sensor name="lidar" type="gpu_lidar">
+      <topic>scan</topic>
+      <gz_frame_id>lidar_link</gz_frame_id>
+      <update_rate>10</update_rate>
+      <always_on>1</always_on>
+      <visualize>true</visualize>
+      <lidar>
+        <scan>
+          <horizontal>
+            <samples>360</samples>
+            <resolution>1</resolution>
+            <min_angle>-3.14159</min_angle>
+            <max_angle>3.14159</max_angle>
+          </horizontal>
+          <vertical>
+            <samples>1</samples>
+            <resolution>1</resolution>
+            <min_angle>0</min_angle>
+            <max_angle>0</max_angle>
+          </vertical>
+        </scan>
+        <range>
+          <min>0.12</min>
+          <max>12.0</max>
+          <resolution>0.01</resolution>
+        </range>
+        <noise>
+          <type>gaussian</type>
+          <mean>0.0</mean>
+          <stddev>0.01</stddev>
+        </noise>
+      </lidar>
+    </sensor>
+  </gazebo>
+  <gazebo reference="imu_link">
+    <sensor name="imu" type="imu">
+      <topic>imu/data</topic>
+      <gz_frame_id>imu_link</gz_frame_id>
+      <update_rate>50</update_rate>
+      <always_on>1</always_on>
+      <imu>
+        <angular_velocity>
+          <x><noise type="gaussian"><mean>0</mean><stddev>0.002</stddev></noise></x>
+          <y><noise type="gaussian"><mean>0</mean><stddev>0.002</stddev></noise></y>
+          <z><noise type="gaussian"><mean>0</mean><stddev>0.002</stddev></noise></z>
+        </angular_velocity>
+        <linear_acceleration>
+          <x><noise type="gaussian"><mean>0</mean><stddev>0.017</stddev></noise></x>
+          <y><noise type="gaussian"><mean>0</mean><stddev>0.017</stddev></noise></y>
+          <z><noise type="gaussian"><mean>0</mean><stddev>0.017</stddev></noise></z>
+        </linear_acceleration>
+      </imu>
+    </sensor>
+  </gazebo>
   <!-- ═══════════════════════════════════════════════════════════════════════
        WHEEL MACRO — Modular, used for all 4 wheels

Commit message: Revert "Feature/phase9 integration"

File: src/rover_simulation/urdf/rover.urdf.xacro (robot description, xacro)
@@ -276,84 +276,4 @@
     <xacro:cylinder_inertia m="0.3" r="0.05" l="0.06"/>
   </link>
-  <!-- ═══════════════════════════════════════════════════════════════════════
-       IMU MOUNT — small module on the chassis, just above centre
-  ═══════════════════════════════════════════════════════════════════════════ -->
-  <joint name="imu_joint" type="fixed">
-    <parent link="base_link"/>
-    <child link="imu_link"/>
-    <origin xyz="0 0 0.07" rpy="0 0 0"/>
-  </joint>
-  <link name="imu_link">
-    <visual>
-      <origin xyz="0 0 0" rpy="0 0 0"/>
-      <geometry>
-        <box size="0.04 0.04 0.02"/>
-      </geometry>
-      <material name="dark_grey"/>
-    </visual>
-    <xacro:box_inertia m="0.05" x="0.04" y="0.04" z="0.02"/>
-  </link>
-  <!-- ═══════════════════════════════════════════════════════════════════════
-       SENSORS — LiDAR + IMU.
-       NOTE: at runtime the simulation loads the rover *inlined* in
-       lunar_terrain.world, which carries its own copies of these sensor
-       blocks. These <gazebo> blocks exist only so a future
-       `xacro rover.urdf.xacro | gz sdf -p -` regeneration stays in sync.
-  ═══════════════════════════════════════════════════════════════════════════ -->
-  <gazebo reference="lidar_link">
-    <sensor name="lidar" type="gpu_lidar">
-      <topic>scan</topic>
-      <gz_frame_id>lidar_link</gz_frame_id>
-      <update_rate>10</update_rate>
-      <always_on>1</always_on>
-      <visualize>true</visualize>
-      <lidar>
-        <scan>
-          <horizontal>
-            <samples>360</samples>
-            <resolution>1</resolution>
-            <min_angle>-3.14159</min_angle>
-            <max_angle>3.14159</max_angle>
-          </horizontal>
-          <vertical>
-            <samples>1</samples>
-            <resolution>1</resolution>
-            <min_angle>0</min_angle>
-            <max_angle>0</max_angle>
-          </vertical>
-        </scan>
-        <range>
-          <min>0.12</min>
-          <max>12.0</max>
-          <resolution>0.01</resolution>
-        </range>
-        <noise>
-          <type>gaussian</type>
-          <mean>0.0</mean>
-          <stddev>0.01</stddev>
-        </noise>
-      </lidar>
-    </sensor>
-  </gazebo>
-  <gazebo reference="imu_link">
-    <sensor name="imu" type="imu">
-      <topic>imu/data</topic>
-      <gz_frame_id>imu_link</gz_frame_id>
-      <update_rate>50</update_rate>
-      <always_on>1</always_on>
-      <imu>
-        <angular_velocity>
-          <x><noise type="gaussian"><mean>0</mean><stddev>0.002</stddev></noise></x>
-          <y><noise type="gaussian"><mean>0</mean><stddev>0.002</stddev></noise></y>
-          <z><noise type="gaussian"><mean>0</mean><stddev>0.002</stddev></noise></z>
-        </angular_velocity>
-        <linear_acceleration>
-          <x><noise type="gaussian"><mean>0</mean><stddev>0.017</stddev></noise></x>
-          <y><noise type="gaussian"><mean>0</mean><stddev>0.017</stddev></noise></y>
-          <z><noise type="gaussian"><mean>0</mean><stddev>0.017</stddev></noise></z>
-        </linear_acceleration>
-      </imu>
-    </sensor>
-  </gazebo>
   <!-- ═══════════════════════════════════════════════════════════════════════
        WHEEL MACRO — Modular, used for all 4 wheels
@@ -465,6 +385,4 @@
       <max_angular_acceleration>2.0</max_angular_acceleration>
       <topic>cmd_vel</topic>
-      <odom_topic>odometry</odom_topic>
-      <tf_topic>tf</tf_topic>
       <frame_id>odom</frame_id>
       <child_frame_id>base_footprint</child_frame_id>
@@ -472,3 +390,9 @@
     </plugin>
   </gazebo>
+  <!-- Joint state publisher: no <joint_name> filter = publishes all joints,
+       avoids entity-resolution failure when spawned from URDF via ros_gz_sim create -->
+  <gazebo>
+    <plugin filename="gz-sim-joint-state-publisher-system"
+            name="gz::sim::systems::JointStatePublisher"/>
+  </gazebo>
 </robot>
